File: eda/kicad_6.0.2/nes_peripheral/nes_peripheral.kicad_sch (KiCad schematic)
At the start: 126 parts, among them J1 CONN_USER, J10 CONN_JOY2, J11 CONN_JOY2_OE_SEL, J12 CONN_JOY1_OE_SEL, J13 CONN_JOY1_FC, J14 CONN_JOY1_FC_COMPATIBLE, J15 CONN_JOY1_MIC, J16 CONN_5V_RESERVE, J17 DB15_Female_JOY1, J18 DB9_Female_JOY1, J19 CONN_SOUND_IO, J2 CONN_GPIO0_DBG, J20 CONN_JOY2_FC, J21 CONN_JOY2_FC_COMPATIBLE, J22 CONN_JOY2_MIC, J23 FC_CONN, J24 CONN_CART_DBG, J25 CONN_CART_DBG, J26 DB15_Female_JOY2, J27 DB9_Female_JOY2, J28 CONN_JOY2_DBGSEL, J29 CONN_JOY1_DBGSEL, J3 CONN_GPIO1_DBG, J30 CONN_GAINSEL, J31 Screw_Terminal_SPK, J32 CONN_SPK, J33 CONN_JOY2_DBG, J34 CONN_JOY1_DBG, J4 Jack_EXT5V, J5 CONN_GPIO0_DBG, J6 CONN_GPIO1_DBG, J7 CONN_CART_OE_SEL, J8 CONN_5VSEL, J9 CONN_JOY1, U1 TXB0104PW, U10 TXB0104PW, U11 TXB0104PW, U12 TXB0104PW, U13 TXB0104PW, U14 TXB0104PW, U15 TXB0104PW, U16 TXB0104PW, U17 4021, U18 4021, U19 MAX98357, U2 TXB0104PW, U20 MAX98357, U3 TXB0104PW, U4 TXB0104PW, U5 TXB0104PW, U6 TXB0104PW, U7 TXB0104PW, U8 TXB0104PW, U9 TXB0104PW

Commit message: feat: max98357のフットプリントを追加
Parts:
- C1, C10, C11, C12, C13, C14, C15, C16, C17, C18, C19, C2, C20, C21, C22, C23, C24, C25, C26, C27, C28, C29, C3, C30, C31, C32, C33, C34, C35, C36, C37, C38, C39, C4, C40, C5, C6, C7, C8, C9: footprint (none) -> Capacitor_SMD:C_0603_1608Metric_Pad1.08x0.95mm_HandSolder
- D1, D2, D3: footprint (none) -> LED_SMD:LED_0603_1608Metric_Pad1.05x0.95mm_HandSolder
- F1: footprint (none) -> Fuse:Fuse_0603_1608Metric_Pad1.05x0.95mm_HandSolder
- J1: footprint (none) -> Connector_PinSocket_2.54mm:PinSocket_2x06_P2.54mm_Vertical
- J10, J30, J9: footprint (none) -> Connector_PinSocket_2.54mm:PinSocket_2x05_P2.54mm_Vertical
- J11, J12, J7, J8: footprint (none) -> Connector_PinSocket_2.54mm:PinSocket_1x03_P2.54mm_Vertical
- J13, J20: footprint (none) -> Connector_PinSocket_2.54mm:PinSocket_2x15_P2.54mm_Vertical; symbol Connector_Generic:Conn_02x15_Top_Bottom -> Connector_Generic:Conn_02x15_Odd_Even
- J14, J21: footprint (none) -> Connector_PinSocket_2.54mm:PinSocket_2x09_P2.54mm_Vertical; symbol Connector_Generic:Conn_02x09_Top_Bottom -> Connector_Generic:Conn_02x09_Odd_Even
- J15, J22, J28, J29: footprint (none) -> Connector_PinSocket_2.54mm:PinSocket_2x01_P2.54mm_Vertical
- J16, J19: footprint (none) -> Connector_PinSocket_2.54mm:PinSocket_2x03_P2.54mm_Vertical
- J17, J26: footprint (none) -> Connector_Dsub:DSUB-15-HD_Female_Horizontal_P2.29x1.98mm_EdgePinOffset9.40mm
- J18: footprint (none) -> Connector_Dsub:DSUB-9_Female_Horizontal_P2.77x2.84mm_EdgePinOffset9.40mm
- J2, J3, J5, J6: footprint (none) -> Connector_PinSocket_2.54mm:PinSocket_1x20_P2.54mm_Vertical
- J24, J25: footprint (none) -> Connector_PinSocket_2.54mm:PinSocket_1x30_P2.54mm_Vertical
- J27: footprint (none) -> Connector_Dsub:DSUB-9_Female_Horizontal_P2.77x2.54mm_EdgePinOffset9.40mm
- J31: footprint (none) -> TerminalBlock:TerminalBlock_bornier-4_P5.08mm
- J32, JP1, JP2, R1, R10, R11, R12, R13, R14, R15, R16, R17, R18, R19, R2, R20, R21, R22, R23, R24, R25, R26, R3, R4, R5, R6, R7, R8, R9: footprint (none) -> Resistor_SMD:R_0603_1608Metric_Pad0.98x0.95mm_HandSolder
- J33, J34: footprint (none) -> Resistor_SMD:R_0603_1608Metric_Pad0.98x0.95mm_HandSolder; symbol Connector_Generic:Conn_02x09_Top_Bottom -> Connector_Generic:Conn_02x09_Odd_Even
- J4: footprint (none) -> OPL_Connector:DCJ3P-14.2X11.0X9.0MM; symbol Connector:Jack-DC -> Connector:Barrel_Jack_Switch
- U17, U18: footprint (none) -> Package_SO:SOIC-16W_5.3x10.2mm_P1.27mm
- U19, U20: footprint (none) -> nes_peripheral:QFN-16_EP_3x3_Pitch0.5mm
Connections:
- net +3V3: now also J33.17 (Pin_17), J34.17 (Pin_17); no longer J33.9 (Pin_9), J34.9 (Pin_9)
- net +5V: now also J13.29 (Pin_29), J14.11 (Pin_11), J14.12 (Pin_12), J14.13 (Pin_13), J14.14 (Pin_14), J20.29 (Pin_29), J21.11 (Pin_11), J21.12 (Pin_12), J21.13 (Pin_13), J21.14 (Pin_14); no longer J13.15 (Pin_15), J14.15 (Pin_15), J14.16 (Pin_16), J14.6 (Pin_6), J14.7 (Pin_7), J20.15 (Pin_15), J21.15 (Pin_15), J21.16 (Pin_16), J21.6 (Pin_6), J21.7 (Pin_7)
- net 5V_JOY1_CLK: now also J13.27 (Pin_27), J13.28 (Pin_28), J14.7 (Pin_7), J14.8 (Pin_8); no longer J13.14 (Pin_14), J13.29 (Pin_29), J14.13 (Pin_13), J14.4 (Pin_4)
- net 5V_JOY1_DO: now also J13.25 (Pin_25), J13.26 (Pin_26), J14.3 (Pin_3), J14.4 (Pin_4); no longer J13.13 (Pin_13), J13.28 (Pin_28), J14.11 (Pin_11), J14.2 (Pin_2)
- net 5V_JOY1_P/~{S}: now also J13.23 (Pin_23), J13.24 (Pin_24), J14.5 (Pin_5), J14.6 (Pin_6); no longer J13.12 (Pin_12), J13.27 (Pin_27), J14.12 (Pin_12), J14.3 (Pin_3)
- net 5V_JOY1_RESERVE: now also J13.3 (Pin_3), J13.4 (Pin_4); no longer J13.17 (Pin_17), J13.2 (Pin_2)
- net 5V_JOY2_CLK: now also J20.27 (Pin_27), J20.28 (Pin_28), J21.7 (Pin_7), J21.8 (Pin_8); no longer J20.14 (Pin_14), J20.29 (Pin_29), J21.13 (Pin_13), J21.4 (Pin_4)
- net 5V_JOY2_DO: now also J20.25 (Pin_25), J20.26 (Pin_26), J21.3 (Pin_3), J21.4 (Pin_4); no longer J20.13 (Pin_13), J20.28 (Pin_28), J21.11 (Pin_11), J21.2 (Pin_2)
- net 5V_JOY2_MICIN: now also J20.3 (Pin_3), J20.4 (Pin_4); no longer J20.17 (Pin_17), J20.2 (Pin_2)
- net 5V_JOY2_P/~{S}: now also J20.23 (Pin_23), J20.24 (Pin_24), J21.5 (Pin_5), J21.6 (Pin_6); no longer J20.12 (Pin_12), J20.27 (Pin_27), J21.12 (Pin_12), J21.3 (Pin_3)
- net GND: now also J13.2 (Pin_2), J14.15 (Pin_15), J14.16 (Pin_16), J20.2 (Pin_2), J21.15 (Pin_15), J21.16 (Pin_16), J33.2 (Pin_2), J33.4 (Pin_4), J33.6 (Pin_6), J33.8 (Pin_8), J34.2 (Pin_2), J34.4 (Pin_4), J34.6 (Pin_6), J34.8 (Pin_8), J4.3; no longer J13.16 (Pin_16), J14.8 (Pin_8), J14.9 (Pin_9), J20.16 (Pin_16), J21.8 (Pin_8), J21.9 (Pin_9), J33.11 (Pin_11), J33.13 (Pin_13), J33.15 (Pin_15), J33.17 (Pin_17), J34.11 (Pin_11), J34.13 (Pin_13), J34.15 (Pin_15), J34.17 (Pin_17)
- net JOY1_3V3_DBG_D1: now also J34.3 (Pin_3); no longer J34.2 (Pin_2)
- net JOY1_3V3_DBG_D2: now also J34.5 (Pin_5); no longer J34.3 (Pin_3)
- net JOY1_3V3_DBG_D3: now also J34.7 (Pin_7); no longer J34.4 (Pin_4)
- net JOY1_3V3_DBG_D4: now also J34.9 (Pin_9); no longer J34.5 (Pin_5)
- net JOY1_3V3_DBG_D5: now also J34.11 (Pin_11); no longer J34.6 (Pin_6)
- net JOY1_3V3_DBG_D6: now also J34.13 (Pin_13); no longer J34.7 (Pin_7)
- net JOY1_3V3_DBG_D7: now also J34.15 (Pin_15); no longer J34.8 (Pin_8)
- net JOY2_3V3_DBG_D1: now also J33.3 (Pin_3); no longer J33.2 (Pin_2)
- net JOY2_3V3_DBG_D2: now also J33.5 (Pin_5); no longer J33.3 (Pin_3)
- net JOY2_3V3_DBG_D3: now also J33.7 (Pin_7); no longer J33.4 (Pin_4)
- net JOY2_3V3_DBG_D4: now also J33.9 (Pin_9); no longer J33.5 (Pin_5)
- net JOY2_3V3_DBG_D5: now also J33.11 (Pin_11); no longer J33.6 (Pin_6)
- net JOY2_3V3_DBG_D6: now also J33.13 (Pin_13); no longer J33.7 (Pin_7)
- net JOY2_3V3_DBG_D7: now also J33.15 (Pin_15); no longer J33.8 (Pin_8)

Commit message: feat: FC_CONNのfootprintを作成
Parts:
- J23: footprint (none) -> nes_peripheral:FC_CONN
Changed lines of the file:
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@@
     (property "Reference" "J23" (id 0) (at 390.525 27.94 0))
     (property "Value" "FC_CONN" (id 1) (at 390.525 30.48 0))
-    (property "Footprint" "" (id 2) (at 389.255 69.85 0)
+    (property "Footprint" "nes_peripheral:FC_CONN" (id 2) (at 389.255 69.85 0)
       (effects (font (size 1.27 1.27)) hide)
     )
@@
     )
     (path "/74b4d553-83e0-4956-bbc1-05dc682e5b5a"
-      (reference "J23") (unit 1) (value "FC_CONN") (footprint "")
+      (reference "J23") (unit 1) (value "FC_CONN") (footprint "nes_peripheral:FC_CONN")
     )
     (path "/515b38b0-91db-4d48-94bf-4f99819ee6ef"
