File: eda/kicad_6.0.2/nes_peripheral/nes_peripheral.kicad_sch (KiCad schematic)
At the start: 117 parts, among them J1 CONN_USER, J10 CONN_JOY2, J11 CONN_JOY2_OE_SEL, J12 CONN_JOY1_OE_SEL, J15 CONN_JOY1_MIC, J16 CONN_5V_RESERVE, J2 CONN_JOY1_FC_COMPATIBLE, J22 CONN_JOY2_MIC, J23 FC_CONN, J24 CONN_CART_DBG, J25 CONN_CART_DBG, J28 CONN_JOY2_DBGSEL, J29 CONN_JOY1_DBGSEL, J3 CONN_JOY2_FC_COMPATIBLE, J30 CONN_GAINSEL, J31 Screw_Terminal_SPK, J33 CONN_JOY2_DBG, J34 CONN_JOY1_DBG, J4 Jack_EXT5V, J7 CONN_CART_OE_SEL, J8 CONN_5VSEL, J9 CONN_JOY1, U1 TXB0104PW, U10 TXB0104PW, U11 TXB0104PW, U12 TXB0104PW, U13 TXB0104PW, U14 TXB0104PW, U15 TXB0104PW, U16 TXB0104PW, U17 4021, U18 4021, U19 MAX98357, U2 TXB0104PW, U20 MAX98357, U3 TXB0104PW, U4 TXB0104PW, U5 TXB0104PW, U6 TXB0104PW, U7 TXB0104PW, U8 TXB0104PW, U9 TXB0104PW

Commit message: fix: I2Sのピン配置を変更
Parts:
- J1: footprint Connector_PinSocket_2.54mm:PinSocket_1x06_P2.54mm_Vertical -> Connector_PinSocket_2.54mm:PinSocket_1x04_P2.54mm_Vertical; symbol Connector_Generic:Conn_01x06 -> Connector_Generic:Conn_01x04
- J33, J34: footprint Connector_PinSocket_2.54mm:PinSocket_2x07_P2.54mm_Vertical -> Connector_PinSocket_2.54mm:PinSocket_2x09_P2.54mm_Vertical
Connections:
- net 3V3_JOY1_CLK: now also JP1.36 (Pin_36); no longer JP2.39 (Pin_39)
- net 3V3_JOY1_DO: now also JP1.34 (Pin_34); no longer JP2.35 (Pin_35)
- net 3V3_JOY1_P/~{S}: now also JP1.35 (Pin_35); no longer JP2.37 (Pin_37)
- net 3V3_JOY1_RESERVE: now also JP1.33 (Pin_33); no longer JP2.33 (Pin_33)
- net 3V3_JOY2_CLK: now also JP2.36 (Pin_36); no longer JP2.40 (Pin_40)
- net 3V3_JOY2_DO: now also JP2.34 (Pin_34); no longer JP2.36 (Pin_36)
- net 3V3_JOY2_MICIN: now also JP2.33 (Pin_33); no longer JP2.34 (Pin_34)
- net 3V3_JOY2_P/~{S}: now also JP2.35 (Pin_35); no longer JP2.38 (Pin_38)
- net 3V3_PA1: now also JP1.25 (Pin_25); no longer JP1.35 (Pin_35)
- net 3V3_PA11: now also JP1.24 (Pin_24); no longer JP1.34 (Pin_34)
- net 3V3_PA12: now also JP1.26 (Pin_26); no longer JP1.36 (Pin_36)
- net 3V3_PA2: now also JP1.23 (Pin_23); no longer JP1.33 (Pin_33)
- net 3V3_PA5: now also JP1.21 (Pin_21); no longer JP1.31 (Pin_31)
- net 3V3_PA6: now also JP1.19 (Pin_19); no longer JP1.27 (Pin_27)
- net 3V3_PA7: now also JP1.20 (Pin_20); no longer JP1.28 (Pin_28)
- net 3V3_PA8: now also JP1.22 (Pin_22); no longer JP1.32 (Pin_32)
- net 3V3_PD1: now also JP1.27 (Pin_27); no longer JP1.37 (Pin_37)
- net 3V3_PD2: now also JP1.31 (Pin_31); no longer JP1.39 (Pin_39)
- net 3V3_PD5: now also JP1.32 (Pin_32); no longer JP1.40 (Pin_40)
- net 3V3_PD6: now also JP1.28 (Pin_28); no longer JP1.38 (Pin_38)
- net CART_OE_IN: now also JP2.39 (Pin_39); no longer JP1.25 (Pin_25)
- net DAC_I2S_BCLK: now also JP1.37 (Pin_37); no longer JP1.19 (Pin_19)
- net DAC_I2S_DIN: now also JP1.38 (Pin_38); no longer JP1.20 (Pin_20)
- net DAC_I2S_LRCLK: now also JP1.39 (Pin_39); no longer JP1.21 (Pin_21)
- net DAC_~{SD_MODE}: now also JP1.40 (Pin_40); no longer JP1.22 (Pin_22)
- net GPIO_0_D20 renamed GPIO_1_D33
- net GPIO_1_D33: now also JP2.38 (Pin_38); no longer JP1.23 (Pin_23)
- net GPIO_0_D21 renamed GPIO_1_D35
- net GPIO_1_D35: now also JP2.40 (Pin_40); no longer JP1.24 (Pin_24)
- net GPIO_0_D23 renamed GPIO_1_D32
- net GPIO_1_D32: now also JP2.37 (Pin_37); no longer JP1.26 (Pin_26)
- removed net USER_GPIO2: J1.5 (Pin_5)
- removed net USER_GPIO3: J1.6 (Pin_6)

Commit message: feat: コントローラの3V3パラレル配線を追加
Parts:
- J33, J34: footprint Connector_PinSocket_2.54mm:PinSocket_2x09_P2.54mm_Vertical -> Connector_PinSocket_2.54mm:PinSocket_1x09_P2.54mm_Vertical; symbol Connector_Generic:Conn_02x09_Odd_Even -> Connector_Generic:Conn_01x09
Connections:
- net +3V3: no longer J33.17 (Pin_17), J34.17 (Pin_17)
- net CART_OE_IN: now also JP2.38 (Pin_38); no longer JP2.39 (Pin_39)
- net GND: now also J33.9 (Pin_9), J34.9 (Pin_9); no longer J33.10 (Pin_10), J33.12 (Pin_12), J33.14 (Pin_14), J33.16 (Pin_16), J33.18 (Pin_18), J33.2 (Pin_2), J33.4 (Pin_4), J33.6 (Pin_6), J33.8 (Pin_8), J34.10 (Pin_10), J34.12 (Pin_12), J34.14 (Pin_14), J34.16 (Pin_16), J34.18 (Pin_18), J34.2 (Pin_2), J34.4 (Pin_4), J34.6 (Pin_6), J34.8 (Pin_8)
- net JOY1_3V3_DBG_D0: now also J34.8 (Pin_8); no longer J34.15 (Pin_15)
- net JOY1_3V3_DBG_D1: now also J34.7 (Pin_7); no longer J34.13 (Pin_13)
- net JOY1_3V3_DBG_D2: now also J34.6 (Pin_6); no longer J34.11 (Pin_11)
- net JOY1_3V3_DBG_D3: now also J34.5 (Pin_5); no longer J34.9 (Pin_9)
- net JOY1_3V3_DBG_D4: now also J34.4 (Pin_4); no longer J34.7 (Pin_7)
- net JOY1_3V3_DBG_D5: now also J34.3 (Pin_3); no longer J34.5 (Pin_5)
- net JOY1_3V3_DBG_D6: now also J34.2 (Pin_2); no longer J34.3 (Pin_3)
- net JOY2_3V3_DBG_D0: now also J33.8 (Pin_8); no longer J33.15 (Pin_15)
- net JOY2_3V3_DBG_D1: now also J33.7 (Pin_7); no longer J33.13 (Pin_13)
- net JOY2_3V3_DBG_D2: now also J33.6 (Pin_6); no longer J33.11 (Pin_11)
- net JOY2_3V3_DBG_D3: now also J33.5 (Pin_5); no longer J33.9 (Pin_9)
- net JOY2_3V3_DBG_D4: now also J33.4 (Pin_4); no longer J33.7 (Pin_7)
- net JOY2_3V3_DBG_D5: now also J33.3 (Pin_3); no longer J33.5 (Pin_5)
- net JOY2_3V3_DBG_D6: now also J33.2 (Pin_2); no longer J33.3 (Pin_3)
- net GPIO_1_D33 renamed GPIO_1_D34
- net GPIO_1_D34: now also JP2.39 (Pin_39); no longer JP2.38 (Pin_38)

Commit message: feat: 音声出力回路をモノラルに変更、配線を修正
Parts:
- removed C38: 0.1u, Capacitor_SMD:C_0603_1608Metric_Pad1.08x0.95mm_HandSolder, symbol Device:C_Small
- removed C39: 10p, Capacitor_SMD:C_0603_1608Metric_Pad1.08x0.95mm_HandSolder, symbol Device:C_Small
- removed R24: 330k, Resistor_SMD:R_0603_1608Metric_Pad0.98x0.95mm_HandSolder, symbol Device:R_Small
- removed U20: MAX98357, nes_peripheral:QFN-16_EP_3x3_Pitch0.5mm, symbol nes_peripheral:MAX98357
- J11, J12: footprint Connector_PinHeader_2.54mm:PinHeader_1x03_P2.54mm_Vertical -> Connector_PinHeader_2.54mm:PinHeader_1x02_P2.54mm_Vertical; symbol Connector_Generic:Conn_01x03 -> Connector_Generic:Conn_01x02
- J30: footprint Connector_PinHeader_2.54mm:PinHeader_2x05_P2.54mm_Vertical -> Connector_PinHeader_2.54mm:PinHeader_2x03_P2.54mm_Vertical; symbol Connector_Generic:Conn_02x05_Odd_Even -> Connector_Generic:Conn_02x03_Odd_Even
- J31: footprint TerminalBlock:TerminalBlock_bornier-4_P5.08mm -> TerminalBlock:TerminalBlock_bornier-2_P5.08mm; symbol Connector:Screw_Terminal_01x04 -> Connector:Screw_Terminal_01x02
Connections:
- net +3V3: now also J30.6 (Pin_6); no longer J30.8 (Pin_8)
- net 3V3_JOY1_P/~{S}: now also JP1.33 (Pin_33); no longer JP1.35 (Pin_35)
- net 3V3_JOY1_RESERVE: now also JP1.35 (Pin_35); no longer JP1.33 (Pin_33)
- net 3V3_JOY2_CLK: now also JP2.38 (Pin_38); no longer JP2.36 (Pin_36)
- net 3V3_JOY2_DO: now also JP2.35 (Pin_35); no longer JP2.34 (Pin_34)
- net 3V3_JOY2_MICIN: now also JP2.37 (Pin_37); no longer JP2.33 (Pin_33)
- net 3V3_JOY2_P/~{S}: now also JP2.39 (Pin_39); no longer JP2.35 (Pin_35)
- net CART_OE_IN: now also JP2.40 (Pin_40); no longer JP2.38 (Pin_38)
- net DAC_I2S_DIN: now also JP1.40 (Pin_40); no longer JP1.38 (Pin_38)
- net DAC_I2S_LRCLK: now also JP1.38 (Pin_38); no longer JP1.39 (Pin_39)
- net DAC_~{SD_MODE}: now also JP1.39 (Pin_39); no longer JP1.40 (Pin_40)
- net GAIN_SLOT: now also J30.4 (Pin_4); no longer J30.1 (Pin_1), J30.5 (Pin_5), J30.7 (Pin_7), J30.9 (Pin_9)
- net GND: now also J30.1 (Pin_1), R26.2; no longer J11.3 (Pin_3), J12.3 (Pin_3), J30.4 (Pin_4), R26.1
- net GPIO_1_D32 renamed GPIO_1_D29
- net GPIO_1_D29: now also JP2.34 (Pin_34); no longer JP2.37 (Pin_37)
- net GPIO_1_D34 renamed GPIO_1_D28
- net GPIO_1_D28: now also JP2.33 (Pin_33); no longer JP2.39 (Pin_39)
- net GPIO_1_D35 renamed GPIO_1_D31
- net GPIO_1_D31: now also JP2.36 (Pin_36); no longer JP2.40 (Pin_40)
- net SPK_OUT_L_N renamed SPK_OUT_N
- net SPK_OUT_L_P renamed SPK_OUT_P
- removed net SPK_OUT_R_N: J31.4 (Pin_4)
- removed net SPK_OUT_R_P: J31.3 (Pin_3)
- new net: J30.5 (Pin_5), R26.1
- no-connect marks 11 -> 10
Other:
- note added: "12dB"
- note added: "15dB"
- note added: "3dB"
- note added: "6dB"
- note added: "OPEN: 9dB"
- note added: "close: 5V Serial open : 3V3 Parallel"
- note removed: "15dB 12dB 9dB 6dB 3dB"
- note removed: "5V Serial 3V3 Parallel"
- moved on the sheet: R25, R26

Commit message: wip: 全部の部品を載せた
Parts:
- removed J10: CONN_JOY2, Connector_PinSocket_2.54mm:PinSocket_1x06_P2.54mm_Vertical, symbol Connector_Generic:Conn_01x06
- removed J9: CONN_JOY1, Connector_PinSocket_2.54mm:PinSocket_1x06_P2.54mm_Vertical, symbol Connector_Generic:Conn_01x06
Connections:
- net GPIO_1_D28: now also J1.4 (Pin_4); no longer J1.3 (Pin_3)
- net GPIO_1_D31: now also J1.3 (Pin_3); no longer J1.4 (Pin_4)
Other:
- note removed: "Joypad 3V3 Serial"
- moved on the sheet: J11, J12, R5, R6

Commit message: feat: コントローラ用回路を引いた
Connections:
- net 3V3_JOY2_CLK: now also U16.2 (A1); no longer U16.4 (A3)
- net 3V3_JOY2_DO: now also JP2.37 (Pin_37), U16.4 (A3); no longer JP2.35 (Pin_35), U16.2 (A1)
- net 3V3_JOY2_MICIN: now also JP2.35 (Pin_35); no longer JP2.37 (Pin_37)
- net 5V_JOY2_CLK: now also U16.13 (B1); no longer U16.11 (B3)
- net 5V_JOY2_DO: now also U16.11 (B3); no longer U16.13 (B1)
Changed lines of the file:
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@@
     (effects (font (size 1.27 1.27)) (justify left bottom))
   )
-  (label "3V3_JOY2_CLK" (at 344.17 282.575 180)
+  (label "3V3_JOY2_CLK" (at 344.17 272.415 180)
     (effects (font (size 1.27 1.27)) (justify right bottom))
   )
@@
     (effects (font (size 1.27 1.27)) (justify right bottom))
   )
-  (label "5V_JOY2_DO" (at 364.49 272.415 0)
+  (label "5V_JOY2_DO" (at 364.49 282.575 0)
     (effects (font (size 1.27 1.27)) (justify left bottom))
   )
@@
     (effects (font (size 1.27 1.27)) (justify right bottom))
   )
-  (label "3V3_JOY2_DO" (at 344.17 272.415 180)
+  (label "3V3_JOY2_DO" (at 344.17 282.575 180)
     (effects (font (size 1.27 1.27)) (justify right bottom))
   )
@@
     (effects (font (size 1.27 1.27)) (justify right bottom))
   )
-  (label "3V3_JOY2_MICIN" (at 52.705 134.62 180)
+  (label "3V3_JOY2_MICIN" (at 52.705 132.08 180)
     (effects (font (size 1.27 1.27)) (justify right bottom))
   )
@@
     (effects (font (size 1.27 1.27)) (justify left bottom))
   )
-  (label "5V_JOY2_CLK" (at 364.49 282.575 0)
+  (label "5V_JOY2_CLK" (at 364.49 272.415 0)
     (effects (font (size 1.27 1.27)) (justify left bottom))
   )
@@
     (effects (font (size 1.27 1.27)) (justify right bottom))
   )
-  (label "3V3_JOY2_DO" (at 52.705 132.08 180)
+  (label "3V3_JOY2_DO" (at 52.705 134.62 180)
     (effects (font (size 1.27 1.27)) (justify right bottom))
   )
@@
   (symbol (lib_id "Connector_Generic:Conn_01x02") (at 283.21 294.005 90) (mirror x) (unit 1)
     (in_bom yes) (on_board yes)
-    (property "Reference" "J15" (id 0) (at 280.162 282.702 90)
+    (property "Reference" "J15" (id 0) (at 289.814 282.829 90)
       (effects (font (size 1.27 1.27)) (justify left))
     )
-    (property "Value" "CONN_JOY1_MIC" (id 1) (at 286.131 284.988 90)
+    (property "Value" "CONN_JOY1_MIC" (id 1) (at 295.783 285.115 90)
       (effects (font (size 1.27 1.27)) (justify left))
     )
@@
   (symbol (lib_id "Connector_Generic:Conn_01x02") (at 381 292.735 90) (mirror x) (unit 1)
     (in_bom yes) (on_board yes)
-    (property "Reference" "J22" (id 0) (at 377.317 282.702 90)
+    (property "Reference" "J22" (id 0) (at 386.334 281.686 90)
       (effects (font (size 1.27 1.27)) (justify left))
     )
-    (property "Value" "CONN_JOY2_MIC" (id 1) (at 382.778 285.242 90)
+    (property "Value" "CONN_JOY2_MIC" (id 1) (at 392.049 284.353 90)
       (effects (font (size 1.27 1.27)) (justify left))
     )

Commit message: feat: LCSCの部品番号を追加
Parts:
- C1, C10, C11, C12, C13, C14, C15, C16, C17, C18, C19, C2, C20, C21, C22, C23, C24, C25, C26, C27, C28, C29, C3, C30, C31, C32, C33, C34, C35, C36, C37, C4, C5, C6, C7, C8, C9: LCSC (none) -> C14663
- C40: LCSC (none) -> C1634
- D1, D2, D3: LCSC (none) -> C99290
- F1: LCSC (none) -> C207010
- R1, R10, R11, R12, R13, R14, R15, R16, R17, R18, R19, R2, R20, R21, R22, R3, R4, R5, R6, R7, R8, R9: LCSC (none) -> C98220
- R23: LCSC (none) -> C95177
- R25, R26: LCSC (none) -> C100048
- U1, U10, U11, U12, U13, U14, U15, U16, U2, U3, U4, U5, U6, U7, U8, U9: LCSC (none) -> C60708
- U17, U18: LCSC (none) -> C233572
- U19: LCSC (none) -> C910544
