File: eda/kicad_6.0.2/nes_peripheral/_autosave-nes_peripheral.kicad_sch (KiCad schematic)
At the start: 117 parts, among them J1 CONN_USER, J10 CONN_JOY2, J11 CONN_JOY2_OE_SEL, J12 CONN_JOY1_OE_SEL, J15 CONN_JOY1_MIC, J16 CONN_5V_RESERVE, J2 CONN_JOY1_FC_COMPATIBLE, J22 CONN_JOY2_MIC, J23 FC_CONN, J24 CONN_CART_DBG, J25 CONN_CART_DBG, J28 CONN_JOY2_DBGSEL, J29 CONN_JOY1_DBGSEL, J3 CONN_JOY2_FC_COMPATIBLE, J30 CONN_GAINSEL, J31 Screw_Terminal_SPK, J33 CONN_JOY2_DBG, J34 CONN_JOY1_DBG, J4 Jack_EXT5V, J7 CONN_CART_OE_SEL, J8 CONN_5VSEL, J9 CONN_JOY1, U1 TXB0104PW, U10 TXB0104PW, U11 TXB0104PW, U12 TXB0104PW, U13 TXB0104PW, U14 TXB0104PW, U15 TXB0104PW, U16 TXB0104PW, U17 4021, U18 4021, U19 MAX98357, U2 TXB0104PW, U20 MAX98357, U3 TXB0104PW, U4 TXB0104PW, U5 TXB0104PW, U6 TXB0104PW, U7 TXB0104PW, U8 TXB0104PW, U9 TXB0104PW

Commit message: wip: 電源配線中
Parts:
- J33, J34: footprint Connector_PinSocket_2.54mm:PinSocket_2x07_P2.54mm_Vertical -> Connector_PinSocket_2.54mm:PinSocket_2x09_P2.54mm_Vertical
Changed lines of the file:
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@@
     (property "Reference" "J34" (id 0) (at 556.514 265.176 0))
     (property "Value" "CONN_JOY1_DBG" (id 1) (at 556.514 267.716 0))
-    (property "Footprint" "Connector_PinSocket_2.54mm:PinSocket_2x07_P2.54mm_Vertical" (id 2) (at 555.244 281.686 0)
+    (property "Footprint" "Connector_PinSocket_2.54mm:PinSocket_2x09_P2.54mm_Vertical" (id 2) (at 555.244 281.686 0)
       (effects (font (size 1.27 1.27)) hide)
     )
@@
     (property "Reference" "J33" (id 0) (at 556.26 327.66 0))
     (property "Value" "CONN_JOY2_DBG" (id 1) (at 556.26 330.2 0))
-    (property "Footprint" "Connector_PinSocket_2.54mm:PinSocket_2x07_P2.54mm_Vertical" (id 2) (at 554.99 344.678 0)
+    (property "Footprint" "Connector_PinSocket_2.54mm:PinSocket_2x09_P2.54mm_Vertical" (id 2) (at 554.99 344.678 0)
       (effects (font (size 1.27 1.27)) hide)
     )
@@
     )
     (path "/655f1b3b-8f04-4735-84ec-2edcae616bf3"
-      (reference "J33") (unit 1) (value "CONN_JOY2_DBG") (footprint "Connector_PinSocket_2.54mm:PinSocket_2x07_P2.54mm_Vertical")
+      (reference "J33") (unit 1) (value "CONN_JOY2_DBG") (footprint "Connector_PinSocket_2.54mm:PinSocket_2x09_P2.54mm_Vertical")
     )
     (path "/2061fd68-fcee-4b43-8c05-63194c3db933"
-      (reference "J34") (unit 1) (value "CONN_JOY1_DBG") (footprint "Connector_PinSocket_2.54mm:PinSocket_2x07_P2.54mm_Vertical")
+      (reference "J34") (unit 1) (value "CONN_JOY1_DBG") (footprint "Connector_PinSocket_2.54mm:PinSocket_2x09_P2.54mm_Vertical")
     )
     (path "/24f48e35-cc03-4a39-93a5-5ae016295ab9"
