File: eda/kicad_6.0.2/nes_peripheral/nes_peripheral.kicad_pcb (KiCad board)
At the start: 2 copper layers, 100 x 100 mm, 113 parts, among them J1 CONN_USER, J10 CONN_JOY2, J11 CONN_JOY2_OE_SEL, J12 CONN_JOY1_OE_SEL, J15 CONN_JOY1_MIC, J16 CONN_5V_RESERVE, J2 CONN_JOY1_FC_COMPATIBLE, J22 CONN_JOY2_MIC, J23 FC_CONN, J24 CONN_CART_DBG, J25 CONN_CART_DBG, J28 CONN_JOY2_DBGSEL, J29 CONN_JOY1_DBGSEL, J3 CONN_JOY2_FC_COMPATIBLE, J30 CONN_GAINSEL, J31 Screw_Terminal_SPK, J33 CONN_JOY2_DBG, J34 CONN_JOY1_DBG, J4 Jack_EXT5V, J7 CONN_CART_OE_SEL, J8 CONN_5VSEL, J9 CONN_JOY1, U1 TXB0104PW, U10 TXB0104PW, U11 TXB0104PW, U12 TXB0104PW, U13 TXB0104PW, U14 TXB0104PW, U15 TXB0104PW, U16 TXB0104PW, U17 4021, U18 4021, U19 MAX98357, U2 TXB0104PW, U3 TXB0104PW, U4 TXB0104PW, U5 TXB0104PW, U6 TXB0104PW, U7 TXB0104PW, U8 TXB0104PW, U9 TXB0104PW

Commit message: wip: 全部の部品を載せた
Parts:
- removed J10: CONN_JOY2, Connector_PinSocket_2.54mm:PinSocket_1x06_P2.54mm_Vertical
- removed J9: CONN_JOY1, Connector_PinSocket_2.54mm:PinSocket_1x06_P2.54mm_Vertical
- C28, C32, C33, C34, R2, R3, R4: moved to B.Cu
- moved C34 170.4 mm to (132.9, 56.4)
- moved R2 109.9 mm to (52.0, 82.3)
- moved R4 105.3 mm to (72.3, 96.3), turned to 90 degrees
- moved D2 96.5 mm to (52.0, 82.3)
- moved C33 89.4 mm to (96.5, 127.0), turned to 90 degrees
- moved C28 85.2 mm to (96.5, 121.9), turned to -90 degrees
- moved R5 83.3 mm to (74.6, 115.1), turned to -90 degrees
- moved C32 74.1 mm to (124.7, 133.0), turned to -90 degrees
- moved R6 57.9 mm to (61.6, 115.2), turned to -90 degrees
- moved R1 56.2 mm to (106.4, 122.2), turned to -90 degrees
- moved D1 53.7 mm to (104.6, 120.4), turned to 90 degrees
- moved J7 32.5 mm to (68.6, 101.6), turned to 90 degrees
- moved J15 28.4 mm to (81.3, 116.8), turned to 180 degrees
- moved J29 27.9 mm to (55.9, 116.8), turned to 180 degrees
- moved C21 26.5 mm to (86.4, 127.0)
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Connections:
- net /GPIO_1_D35 renamed /CART_OE_IN
- J1 pad 3: /GPIO_1_D28 -> /GPIO_1_D31
- J1 pad 4: /GPIO_1_D31 -> /GPIO_1_D28
Routing:
- net GND: track 3236.3 -> 3216.7 mm
- net /3V3_JOY2_DO: track 0.00 -> 13.8 mm
- net /5V_JOY1_RESERVE: track 12.0 -> 0.00 mm
- net +3V3: track 256.0 -> 244.9 mm, vias 28 -> 26
- net /3V3_JOY2_MICIN: track 0.00 -> 10.3 mm
- net /GPIO_1_D31: track 7.89 -> 17.1 mm
- net /3V3_JOY2_CLK: track 0.00 -> 8.76 mm
- net /CART_OE_IN: track 0.00 -> 8.67 mm
- net /GPIO_1_D29: track 14.1 -> 6.17 mm
- net /3V3_JOY2_P/~{S}: track 0.00 -> 6.45 mm
- net /JOY1_OE_5V: track 6.23 -> 0.00 mm
- net /GPIO_1_D28: track 16.0 -> 21.7 mm
- net /CART_OE: track 129.3 -> 134.2 mm
- net Net-(J29-Pad1): track 21.4 -> 17.7 mm
- net +5V: track 223.0 -> 226.5 mm, vias 19 -> 18
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